File: pcb/corne-cherry.sch (KiCad schematic (older format))
At the start: 87 parts, among them J1 MJ-4PP-9, J2 OLED, J3 LED, P1 i2c-pin, P2 i2c-pin, SW1 SW_PUSH, SW10 SW_PUSH, SW11 SW_PUSH, SW12 SW_PUSH, SW13 SW_PUSH, SW14 SW_PUSH, SW15 SW_PUSH, SW16 SW_PUSH, SW17 SW_PUSH, SW18 SW_PUSH, SW19 SW_PUSH, SW2 SW_PUSH, SW20 SW_PUSH, SW21 SW_PUSH, SW3 SW_PUSH, SW4 SW_PUSH, SW5 SW_PUSH, SW6 SW_PUSH, SW7 SW_PUSH, SW8 SW_PUSH, SW9 SW_PUSH, U1 ProMicro

Commit message: removed corne classic and replaced with corne cherry
Parts:
- JP1: footprint kbd:JP -> kbd:JPC2
- renumbered L7 to L1, L16 to L10, L17 to L11, L18 to L12, L19 to L13, L20 to L14, L21 to L15, L22 to L16, L23 to L17, L24 to L18, L25 to L19, L8 to L2, L26 to L20, L27 to L21, L1 to L22, L2 to L23, L3 to L24, L4 to L25, L5 to L26, L6 to L27, L9 to L3, L10 to L4, L11 to L5, L12 to L6, L13 to L7, L14 to L8, L15 to L9
